File: REgulated Voltage and High Amper supply module.kicad_pcb (KiCad board)
At the start: 2 copper layers, 11 parts, among them J1 IN, 8V-32V, J2 OUT 1,25V -28V, U1 XL4015

Commit message: Regulated Voltage and High Amper supply Module is renewed
Changed lines of the file:
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@@
   )
   (paper "A4")
+  (title_block
+    (title "Regulated Voltage and High Amper Supply Module ")
+    (date "17.11.2022")
+    (rev "1.0")
+    (company "by Muxtar_Safarov")
+  )
   (layers
     (0 "F.Cu" signal)
@@
     (pad_to_mask_clearance 0)
     (pcbplotparams
-      (layerselection 0x00010fc_ffffffff)
+      (layerselection 0x00000e0_ffffffff)
       (plot_on_all_layers_selection 0x0000000_00000000)
       (disableapertmacros false)
@@
       (sketchpadsonfab false)
       (subtractmaskfromsilk false)
-      (outputformat 1)
+      (outputformat 4)
       (mirror false)
-      (drillshape 1)
+      (drillshape 0)
       (scaleselection 1)
-      (outputdirectory "")
+      (outputdirectory "C:/Users/mitxar/Documents/uc3843/microphone MC33063 NE5532/REgulated Voltage and High Amper supply module/")
     )
   )
@@
     (fp_line (start 5.625 5) (end 4.625 5)
       (stroke (width 0.1) (type solid)) (layer "F.Fab"))
-    (pad "1" smd roundrect (at -7.65 -3.4 90) (size 4.6 1.1) (layers "F.Cu" "F.Paste" "F.Mask") (roundrect_rratio 0.227273)
+    (pad "1" smd roundrect (at -7.65 -3.4 90) (size 4.6 1.1) (layers "F.Cu" "F.Paste" "F.Mask") (roundrect_rratio 0.2272727273)
       (net 2 "Earth") (pinfunction "GND") (pintype "power_in"))
-    (pad "2" smd roundrect (at -7.65 -1.7 90) (size 4.6 1.1) (layers "F.Cu" "F.Paste" "F.Mask") (roundrect_rratio 0.227273)
+    (pad "2" smd roundrect (at -7.65 -1.7 90) (size 4.6 1.1) (layers "F.Cu" "F.Paste" "F.Mask") (roundrect_rratio 0.2272727273)
       (net 6 "Net-(U1-FB)") (pinfunction "FB") (pintype "input"))
-    (pad "3" smd roundrect (at -7.65 0 90) (size 4.6 1.1) (layers "F.Cu" "F.Paste" "F.Mask") (roundrect_rratio 0.227273)
-      (net 5 "Net-(D1-K)") (pinfunction "SW") (pintype "power_out"))
-    (pad "3" smd roundrect (at -0.925 -2.775 90) (size 4.55 5.25) (layers "F.Cu" "F.Paste") (roundrect_rratio 0.054945)
-      (net 5 "Net-(D1-K)") (pinfunction "SW") (pintype "power_out"))
-    (pad "3" smd roundrect (at -0.925 2.775 90) (size 4.55 5.25) (layers "F.Cu" "F.Paste") (roundrect_rratio 0.054945)
-      (net 5 "Net-(D1-K)") (pinfunction "SW") (pintype "power_out"))
-    (pad "3" smd roundrect (at 1.5 0 90) (size 9.4 10.8) (layers "F.Cu" "F.Mask") (roundrect_rratio 0.026596)
-      (net 5 "Net-(D1-K)") (pinfunction "SW") (pintype "power_out"))
-    (pad "3" smd roundrect (at 3.925 -2.775 90) (size 4.55 5.25) (layers "F.Cu" "F.Paste") (roundrect_rratio 0.054945)
-      (net 5 "Net-(D1-K)") (pinfunction "SW") (pintype "power_out"))
-    (pad "3" smd roundrect (at 3.925 2.775 90) (size 4.55 5.25) (layers "F.Cu" "F.Paste") (roundrect_rratio 0.054945)
-      (net 5 "Net-(D1-K)") (pinfunction "SW") (pintype "power_out"))
-    (pad "4" smd roundrect (at -7.65 1.7 90) (size 4.6 1.1) (layers "F.Cu" "F.Paste" "F.Mask") (roundrect_rratio 0.227273)
+    (pad "3" smd roundrect (at -7.65 0 90) (size 4.6 1.1) (layers "F.Cu" "F.Paste" "F.Mask") (roundrect_rratio 0.2272727273)
+      (net 5 "Net-(D1-K)") (pinfunction "SW") (pintype "power_out"))
+    (pad "3" smd roundrect (at -0.925 -2.775 90) (size 4.55 5.25) (layers "F.Cu" "F.Paste") (roundrect_rratio 0.05494505495)
+      (net 5 "Net-(D1-K)") (pinfunction "SW") (pintype "power_out"))
+    (pad "3" smd roundrect (at -0.925 2.775 90) (size 4.55 5.25) (layers "F.Cu" "F.Paste") (roundrect_rratio 0.05494505495)
+      (net 5 "Net-(D1-K)") (pinfunction "SW") (pintype "power_out"))
+    (pad "3" smd roundrect (at 1.5 0 90) (size 9.4 10.8) (layers "F.Cu" "F.Mask") (roundrect_rratio 0.02659595745)
+      (net 5 "Net-(D1-K)") (pinfunction "SW") (pintype "power_out"))
+    (pad "3" smd roundrect (at 3.925 -2.775 90) (size 4.55 5.25) (layers "F.Cu" "F.Paste") (roundrect_rratio 0.05494505495)
+      (net 5 "Net-(D1-K)") (pinfunction "SW") (pintype "power_out"))
+    (pad "3" smd roundrect (at 3.925 2.775 90) (size 4.55 5.25) (layers "F.Cu" "F.Paste") (roundrect_rratio 0.05494505495)
+      (net 5 "Net-(D1-K)") (pinfunction "SW") (pintype "power_out"))
+    (pad "4" smd roundrect (at -7.65 1.7 90) (size 4.6 1.1) (layers "F.Cu" "F.Paste" "F.Mask") (roundrect_rratio 0.2272727273)
       (net 4 "Net-(U1-VC)") (pinfunction "VC") (pintype "input"))
-    (pad "5" smd roundrect (at -7.65 3.4 90) (size 4.6 1.1) (layers "F.Cu" "F.Paste" "F.Mask") (roundrect_rratio 0.227273)
+    (pad "5" smd roundrect (at -7.65 3.4 90) (size 4.6 1.1) (layers "F.Cu" "F.Paste" "F.Mask") (roundrect_rratio 0.2272727273)
       (net 3 "VCC") (pinfunction "VIN") (pintype "power_in"))
     (model "${KICAD6_3DMODEL_DIR}/Package_TO_SOT_SMD.3dshapes/TO-263-5_TabPin3.wrl"
