File: REgulated Voltage and High Amper supply module.kicad_sch (KiCad schematic)
At the start: 11 parts, among them J1 IN, 8V-32V, J2 OUT 1,25V -28V, U1 XL4015

Commit message: Regulated Voltage and High Amper supply Module is renewed
Other:
- company: (none) -> by Muxtar_Safarov
- title: (none) -> Regulated Voltage and High Amper Supply Mode 
Changed lines of the file:
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@@
 (kicad_sch (version 20230121) (generator eeschema)
   (paper "A4")
+  (title_block
+    (title "Regulated Voltage and High Amper Supply Mode ")
+    (date "17.11.2022")
+    (rev "1.0")
+    (company "by Muxtar_Safarov")
+  )
   (junction (at 215.9 73.66) (diameter 0) (color 0 0 0 0)
   )
